File: HARDWARE/Relay Wifi.kicad_sch (KiCad schematic)
At the start: 42 parts, among them J1 Bornera 01x02, J10 Screw_Terminal_01x03, J11 HC-SR04, J12 Conn_01x02_Pin, J2 Screw_Terminal_01x03, J3 Screw_Terminal_01x03, J4 Screw_Terminal_01x03, J5 Screw_Terminal_01x03, J6 Screw_Terminal_01x03, J7 Screw_Terminal_01x03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

Commit message: Actualizo el esquematico
Parts:
- removed J12: Conn_01x02_Pin, EESTN5:Jumper, symbol Connector:Conn_01x02_Pin
- added Switch: SW_SPDT, EESTN5:Pin_Header_3, symbol EESTN5:SW_SPDT
Connections:
- net VCC: now also Switch.3 (C); no longer J1.1 (Pin_1)
- new net BAT: J1.1 (Pin_1), Switch.2 (B)
- no-connect marks 0 -> 29
Other:
- moved on the sheet: J1

Commit message: Agrego carpeta hardware con archivos
Parts:
- removed J10, J2, J3, J4, J5, J6, J7, J8: Screw_Terminal_01x03, TerminalBlock:TerminalBlock_bornier-3_P5.08mm, symbol Connector:Screw_Terminal_01x03
- added J12, J2, J3, J4: Screw_Terminal_01x04, TerminalBlock_Altech:Altech_AK100_1x04_P5.00mm, symbol Connector:Screw_Terminal_01x04
- Q1, Q2, Q3, Q4: footprint EESTN5:to92 -> EESTN5:SOT23
- U2, U3, U5, U6: footprint Package_DIP:DIP-4_W7.62mm -> EESTN5:DIP-4_PC817
- U4: footprint Package_TO_SOT_THT:TO-220-3_Vertical -> Package_TO_SOT_SMD:TO-263-3_TabPin2
- renumbered Switch to Switch1
Connections:
- net ECHO: now also U1.7 (IO32); no longer U1.4 (SVN)
- net TRIGGER: now also U1.8 (IO33); no longer U1.9 (IO25)
- net com1: now also J12.1 (Pin_1)
- net com2: now also J12.4 (Pin_4)
- net com3: now also J2.1 (Pin_1)
- net com4: now also J2.4 (Pin_4)
- net com5: now also J3.1 (Pin_1)
- net com6: now also J3.4 (Pin_4)
- net com7: now also J4.1 (Pin_1)
- net com8: now also J4.4 (Pin_4)
- net relay_1: now also U1.31 (IO19); no longer U1.6 (IO35)
- net relay_2: now also U1.30 (IO18); no longer U1.5 (IO34)
- net relay_3: now also U1.28 (IO17); no longer U1.7 (IO32)
- net relay_4: now also U1.27 (IO16); no longer U1.8 (IO33)
- net at K1.9: now also J2.3 (Pin_3)
- net at K3.8: now also J12.2 (Pin_2)
- net at K4.9: now also J4.3 (Pin_3)
- net at K2.9: now also J3.3 (Pin_3)
- net at K4.8: now also J4.2 (Pin_2)
- net at K1.8: now also J2.2 (Pin_2)
- net at K3.9: now also J12.3 (Pin_3)
- net at K2.8: now also J3.2 (Pin_2)
- no-connect marks 29 -> 37
Other:
- note added: "SENSORES"
- moved on the sheet: J11, J9, R1, R4

Commit message: Agrego el nuevo diseño de la placa y el esquematico
Parts:
- added C3: C, Capacitor_SMD:CP_Elec_10x10, symbol Device:C
- D2, D4, D7, D8: footprint Diode_SMD:D_0805_2012Metric_Pad1.15x1.40mm_HandSolder -> Diode_SMD:D_SMA
- Switch1: footprint EESTN5:Pin_Header_3 -> TerminalBlock:TerminalBlock_bornier-3_P5.08mm
Connections:
- net +5V: now also C3.1
- net GND: now also C3.2
Changed lines of the file:
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@@
 	)
 	(junction
+		(at 99.06 53.34)
+		(diameter 0)
+		(color 0 0 0 0)
+	)
+	(junction
 		(at 76.2 40.64)
 		(diameter 0)
@@
 	(wire
 		(pts
+			(xy 107.95 43.18) (xy 107.95 40.64)
+		)
+		(stroke
+			(width 0)
+			(type default)
+		)
+	)
+	(wire
+		(pts
 			(xy 231.14 181.61) (xy 231.14 189.23)
 		)
@@
 	(wire
 		(pts
+			(xy 107.95 53.34) (xy 99.06 53.34)
+		)
+		(stroke
+			(width 0)
+			(type default)
+		)
+	)
+	(wire
+		(pts
 			(xy 100.965 95.25) (xy 100.965 95.885)
 		)
@@
 	(wire
 		(pts
+			(xy 107.95 40.64) (xy 99.06 40.64)
+		)
+		(stroke
+			(width 0)
+			(type default)
+		)
+	)
+	(wire
+		(pts
 			(xy 206.375 219.075) (xy 215.265 219.075)
 		)
@@
 	(wire
 		(pts
+			(xy 107.95 50.8) (xy 107.95 53.34)
+		)
+		(stroke
+			(width 0)
+			(type default)
+		)
+	)
+	(wire
+		(pts
 			(xy 144.145 120.015) (xy 146.685 120.015)
 		)
@@
 			)
 		)
-		(property "Footprint" "Diode_SMD:D_0805_2012Metric_Pad1.15x1.40mm_HandSolder"
+		(property "Footprint" "Diode_SMD:D_SMA"
 			(at 109.22 250.19 0)
 			(effects
@@
 			)
 		)
-		(property "Footprint" "Diode_SMD:D_0805_2012Metric_Pad1.15x1.40mm_HandSolder"
+		(property "Footprint" "Diode_SMD:D_SMA"
 			(at 223.52 250.19 0)
 			(effects
@@
 			)
 		)
-		(property "Footprint" "EESTN5:Pin_Header_3"
+		(property "Footprint" "TerminalBlock:TerminalBlock_bornier-3_P5.08mm"
 			(at 47.625 60.325 0)
 			(effects
@@
 	)
 	(symbol
+		(lib_id "Device:C")
+		(at 107.95 46.99 0)
+		(unit 1)
+		(exclude_from_sim no)
+		(in_bom yes)
+		(on_board yes)
+		(dnp no)
+		(fields_autoplaced yes)
+		(property "Reference" "C3"
+			(at 111.76 45.7199 0)
+			(effects
+				(font
+					(size 1.27 1.27)
+				)
+				(justify left)
+			)
+		)
+		(property "Value" "C"
+			(at 111.76 48.2599 0)
+			(effects
+				(font
+					(size 1.27 1.27)
+				)
+				(justify left)
+			)
+		)
+		(property "Footprint" "Capacitor_SMD:CP_Elec_10x10"
+			(at 108.9152 50.8 0)
+			(effects
+				(font
+					(size 1.27 1.27)
+				)
+				(hide yes)
+			)
+		)
+		(property "Datasheet" "~"
+			(at 107.95 46.99 0)
+			(effects
+				(font
+					(size 1.27 1.27)
+				)
+				(hide yes)
+			)
+		)
+		(property "Description" "Unpolarized capacitor"
+			(at 107.95 46.99 0)
+			(effects
+				(font
+					(size 1.27 1.27)
+				)
+				(hide yes)
+			)
+		)
+		(pin "1"
+		)
+		(pin "2"
+		)
+		(instances
+			(project ""
+				(path "/162603eb-7778-4005-b9b4-324e6481b3d0"
+					(reference "C3")
+					(unit 1)
+				)
+			)
+		)
+	)
+	(symbol
 		(lib_id "power:GND")
 		(at 138.43 87.63 0)
@@
 			)
 		)
-		(property "Footprint" "Diode_SMD:D_0805_2012Metric_Pad1.15x1.40mm_HandSolder"
+		(property "Footprint" "Diode_SMD:D_SMA"
 			(at 223.52 193.675 0)
 			(effects
@@
 			)
 		)
-		(property "Footprint" "Diode_SMD:D_0805_2012Metric_Pad1.15x1.40mm_HandSolder"
+		(property "Footprint" "Diode_SMD:D_SMA"
 			(at 109.22 193.675 0)
 			(effects
